Commit message: 意外修改，目前已经复原

File: src/holosoma_retargeting/holosoma_retargeting/models/mushroom/mushroom_static.urdf (robot description, URDF)
Before this commit: robot mushroom, 1 links, 0 joints
Links:
- link mushroom_link: geometry collision mesh filename=mushroom_visual.obj scale=1 1 1; visual mesh filename=mushroom_visual.obj scale=1 1 1
